File: pcb/lunakbd.kicad_pcb (KiCad board)
At the start: 2 copper layers, 134.4 x 112.7 mm, 64 parts, among them J1 TRRS-PJ-320D, J2 Battery_Socket, J3 Conn_Display, SW1 Switch, SW10 Switch, SW11 Switch, SW12 Switch, SW13 Switch, SW14 Switch, SW15 Switch, SW16 Switch, SW17 Switch, SW18 Switch, SW19 Switch, SW2 Switch, SW20 Switch, SW21 Switch, SW22 Switch, SW23 Switch, SW24 Switch, SW25 Switch, SW26 Switch, SW27 Switch, SW28 Switch, SW29 RotaryEncoder_SW, SW3 Switch, SW30 Reset_Button, SW31 Battery_Switch, SW4 Switch, SW5 Switch, SW6 Switch, SW7 Switch, SW8 Switch, SW9 Switch, U1 ProMicro

Commit message: feat: make all footprints inversibles
Parts:
- D1, D10, D11, D12, D13, D14, D15, D16, D17, D18, D19, D2, D20, D21, D22, D23, D24, D25, D26, D27, D28, D29, D3, D4, D5, D6, D7, D8, D9: footprint Diode_SMD:D_SOD-123 -> Library:D_SOD-123
- J1: footprint Keebio-Parts:TRRS-PJ-320D -> Library:TRRS-PJ-320D
- SW1, SW10, SW11, SW12, SW13, SW14, SW15, SW16, SW17, SW18, SW19, SW2, SW20, SW21, SW22, SW23, SW24, SW25, SW26, SW27, SW3, SW4, SW5, SW6, SW7, SW8, SW9: footprint PCM_Switch_Keyboard_Hotswap_Kailh:SW_Hotswap_Kailh_MX_1.00u -> Library:SW_Hotswap_Kailh_MX_1.00u
- SW28: footprint PCM_Switch_Keyboard_Hotswap_Kailh:SW_Hotswap_Kailh_MX_1.25u_90deg -> Library:SW_Hotswap_Kailh_MX_1.25u_90deg
- SW30: footprint kbd:SW_TL3330AF130QG -> Library:SW_TL3330AF130QG
- SW31: footprint PCM_marbastlib-various:SW_MSK12C02-HB -> Library:SW_MSK12C02-HB
Routing:
- net row-4: vias 0 -> 5
- net row-3: vias 0 -> 6
- net row-2: vias 0 -> 6
- net row-1: vias 0 -> 6
- net row-0: vias 0 -> 6
- net reset: vias 0 -> 1
- net Net-(D9-A): vias 0 -> 1
- net Net-(D8-A): vias 0 -> 1
- net Net-(D7-A): vias 0 -> 1
- net Net-(D6-A): vias 0 -> 1
- net Net-(D5-A): vias 0 -> 1
- net Net-(D4-A): vias 0 -> 1
- net Net-(D3-A): vias 0 -> 1
- net Net-(D29-A): vias 0 -> 1
- net Net-(D28-A): vias 0 -> 1
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
Commit message: feat: trace routes
Connections:
- SW30 pad 1: reset -> GND
- SW30 pad 2: GND -> reset
Routing:
- net col-1: track 0.00 -> 233.8 mm, vias 0 -> 6
- net col-0: track 0.00 -> 213.6 mm, vias 0 -> 5
- net col-2: track 0.00 -> 201.0 mm, vias 0 -> 6
- net col-3: track 0.00 -> 197.3 mm, vias 0 -> 9
- net col-4: track 0.00 -> 185.8 mm, vias 0 -> 7
- net col-5: track 0.00 -> 169.4 mm, vias 0 -> 5
- net row-4: track 0.00 -> 152.8 mm, vias 5 -> 0
- net row-3: track 0.00 -> 146.2 mm, vias 6 -> 0
- net row-2: track 0.00 -> 129.5 mm, vias 6 -> 0
- net row-1: track 0.00 -> 113.2 mm, vias 6 -> 0
- net row-0: track 0.00 -> 109.0 mm, vias 6 -> 0
- net enc-b: track 0.00 -> 62.4 mm, vias 0 -> 3
- net enc-a: track 0.00 -> 60.8 mm, vias 0 -> 3
- net data: track 0.00 -> 54.6 mm, vias 0 -> 1
- net VCC: track 0.00 -> 49.5 mm, vias 0 -> 2
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Other:
- outline, holes or cut-outs redrawn
