File: pcb/lunakbd.kicad_sch (KiCad schematic)
At the start: 72 parts, among them J1 TRRS-PJ-320D, J2 Battery_Socket, J3 Conn_Display, SW1 Switch, SW10 Switch, SW11 Switch, SW12 Switch, SW13 Switch, SW14 Switch, SW15 Switch, SW16 Switch, SW17 Switch, SW18 Switch, SW19 Switch, SW2 Switch, SW20 Switch, SW21 Switch, SW22 Switch, SW23 Switch, SW24 Switch, SW25 Switch, SW26 Switch, SW27 Switch, SW28 Switch, SW29 RotaryEncoder_SW, SW3 Switch, SW30 Reset_Button, SW31 Battery_Switch, SW4 Switch, SW5 Switch, SW6 Switch, SW7 Switch, SW8 Switch, SW9 Switch, U1 ProMicro

Commit message: fix: clearence errors
Parts:
- SW30: footprint lunalib:SW_TL3330AF130QG -> lunalib:SW-SMD_SHOU_TS36CA-0.6
Connections:
- net GND: now also SW30.2; no longer SW30.1
- net reset: now also SW30.1; no longer SW30.2
Changed lines of the file:
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@@
 		(lib_id "Switch:SW_Push")
 		(at 58.42 86.36 0)
-		(mirror y)
 		(unit 1)
 		(exclude_from_sim no)
@@
 			)
 		)
-		(property "Footprint" "lunalib:SW_TL3330AF130QG"
+		(property "Footprint" "lunalib:SW-SMD_SHOU_TS36CA-0.6"
 			(at 58.42 81.28 0)
 			(effects
